Commit message: Prepare new features for part1 of the project

File: install/barista_robot_description/share/barista_robot_description/urdf/barista_robot_model.urdf (robot description, URDF)
Before this commit: robot barista_bot, 16 links, 15 joints
Links:
- link lidar: mass 1 -> None; geometry visual mesh filename=package://barista_robot_description/meshes/hokuyo_urg_04lx.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 scale=0.5 0.5 0.5
